Commit message: revised hokuyo mass

File: hector_gazebo_src/hector_sensors_description/urdf/hokuyo_utm30lx.urdf.xacro (robot description, xacro)
@@ -10,5 +10,5 @@
       <link name="${name}_frame">
         <inertial>
-          <mass value="0.270" />
+          <mass value="0.000270" />
           <origin xyz="0 0 0" rpy="0 0 0" />
           <inertia ixx="2.632e-4" ixy="0" ixz="0" iyy="2.632e-4" iyz="0" izz="1.62e-4" />
